File: KiCAD/BackPanel/BackPanel.kicad_pcb (KiCad board)
At the start: 2 copper layers, 71 x 25 mm, 7 parts

Commit message: Add fabrication notes to indicate where to place production codes.
Other:
- board text added: "Please place Production Code here on back silkscreen."
Changed lines of the file:
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@@
   (general
     (thickness 1.6)
-    (drawings 27)
+    (drawings 30)
     (tracks 0)
     (zones 0)
@@
     (visible_elements FFFFFF7F)
     (pcbplotparams
-      (layerselection 0x010f0_ffffffff)
+      (layerselection 0x110f0_ffffffff)
       (usegerberextensions false)
       (usegerberattributes false)
@@
       (net 1 GND))
   )
+  (gr_text "Please place Production Code here on back silkscreen." (at 159.5 71.75) (layer B.Fab)
+    (effects (font (size 1 1) (thickness 0.15)) (justify mirror))
+  )
+  (gr_line (start 156.5 76.75) (end 159.25 72.5) (layer B.Fab) (width 0.15))
+  (gr_circle (center 155.25 77.75) (end 156.75 77.5) (layer B.Fab) (width 0.15))
   (gr_text "Rev B" (at 114.5 97) (layer B.SilkS)
     (effects (font (size 3 3) (thickness 0.15)) (justify mirror))
