File: KiCAD/FrontPanel/FrontPanel.kicad_pcb (KiCad board)
At the start: 2 copper layers, 71 x 25 mm, 9 parts

Commit message: Add fabrication notes to indicate where to place production codes.
Other:
- board text added: "Please place Production Code here on back silkscreen."
Changed lines of the file:
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@@
   (general
     (thickness 1.6)
-    (drawings 18)
+    (drawings 21)
     (tracks 0)
     (zones 0)
@@
     (visible_elements FFFFFF7F)
     (pcbplotparams
-      (layerselection 0x010f1_ffffffff)
+      (layerselection 0x110f0_ffffffff)
       (usegerberextensions false)
       (usegerberattributes false)
@@
     (pad 1 np_thru_hole circle (at 0 0) (size 3.5 3.5) (drill 3.5) (layers *.Cu *.Mask))
   )
+  (gr_text "Please place Production Code here on back silkscreen." (at 156 72) (layer B.Fab)
+    (effects (font (size 1 1) (thickness 0.15)) (justify mirror))
+  )
+  (gr_line (start 154.5 76.5) (end 156.5 73) (layer B.Fab) (width 0.15))
+  (gr_circle (center 153.5 77.75) (end 154.75 78.5) (layer B.Fab) (width 0.15))
   (dimension 7.75 (width 0.12) (layer Dwgs.User)
     (gr_text "7.750 mm" (at 91.73 96.625 270) (layer Dwgs.User)
