File: KiCAD/Spacer/Spacer.kicad_pcb (KiCad board)
At the start: 2 copper layers, 21 x 4 mm, 0 parts

Commit message: Add fabrication notes to indicate where to place production codes.
Other:
- board text added: "Please place Production Code here on front silkscreen."
Changed lines of the file:
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@@
   (general
     (thickness 1.6)
-    (drawings 13)
+    (drawings 17)
     (tracks 0)
     (zones 0)
@@
     (visible_elements FFFFFF7F)
     (pcbplotparams
-      (layerselection 0x010f0_7ffffffe)
+      (layerselection 0x210e0_7ffffffe)
       (usegerberextensions false)
       (usegerberattributes false)
@@
     (uvia_drill 0.1)
   )
+  (gr_text "Please place Production Code here on front silkscreen." (at 164 81.75) (layer F.Fab)
+    (effects (font (size 1 1) (thickness 0.15)))
+  )
+  (gr_line (start 164 82.5) (end 165.25 82.5) (layer F.Fab) (width 0.15))
+  (gr_line (start 161.5 84.5) (end 164 82.5) (layer F.Fab) (width 0.15))
+  (gr_circle (center 161 84.75) (end 161 85.25) (layer F.Fab) (width 0.15))
   (dimension 18 (width 0.15) (layer Dwgs.User)
     (gr_text "18.000 mm" (at 160.5 92.05) (layer Dwgs.User)
