File: PCB/KiCAD/Nucleo32TNC.kicad_pcb (KiCad board)
At the start: 2 copper layers, 66 x 99 mm, 54 parts, among them J1 AudioJack4, Q1 2N7000, Q2 2N7000, SW1 SW_Push, U1 MCP6004, U2 24LC32

Commit message: Update footprints in schematic, and values for J1 and SW1 in schematic and PCB.  Add an interactive BOM.  Update the README.
Parts:
- J1: value AudioJack4 -> SJ-43515TS
- SW1: value SW_Push -> PTS645VL58-2 LFS
Changed lines of the file:
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@@
       (effects (font (size 1 1) (thickness 0.15)))
     )
-    (fp_text value SW_Push (at 2.25 5.38988) (layer F.Fab)
+    (fp_text value "PTS645VL58-2 LFS" (at 2.25 5.38988) (layer F.Fab)
       (effects (font (size 1 1) (thickness 0.15)))
     )
@@
       (effects (font (size 0.480623 0.480623) (thickness 0.015)))
     )
-    (fp_text value AudioJack4 (at -0.482843 6.195715 90) (layer F.Fab)
+    (fp_text value SJ-43515TS (at -0.482843 6.195715 90) (layer F.Fab)
       (effects (font (size 0.48004 0.48004) (thickness 0.015)))
     )
